File: mxnatee_bot_plate.kicad_pcb (KiCad board)
At the start: 2 copper layers, 137.5 x 139.4 mm, 8 parts, among them U4 HOLE

Commit message: uh did stuff
Parts:
- removed the U4 at (103.8, 35.1)
- removed the U4 at (122.8, 98.4)
- removed the U4 at (129.2, 145.5)
- removed the U4 at (70.7, 106.2)
- removed the U4 at (44.1, 91.1)
- added U4: HOLE, Keybage_MountingHoles:MountingHole_2.2mm_M2_Pad_NoSilk, F.Cu at (103.8, 35.1)
- added U4: HOLE, Keybage_MountingHoles:MountingHole_2.2mm_M2_Pad_NoSilk, F.Cu at (122.8, 98.4)
- added U4: HOLE, Keybage_MountingHoles:MountingHole_2.2mm_M2_Pad_NoSilk, F.Cu at (129.2, 145.5)
- added U4: HOLE, Keybage_MountingHoles:MountingHole_2.2mm_M2_Pad_NoSilk, F.Cu at (70.7, 106.2)
- added U4: HOLE, Keybage_MountingHoles:MountingHole_2.2mm_M2_Pad_NoSilk, F.Cu at (44.1, 91.1)
- U4: footprint Keebio-Parts:MountingHole -> Keybage_MountingHoles:MountingHole_2.2mm_M2_Pad_NoSilk
Changed lines of the file:
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@@
     (uvia_drill 0.1)
+  )
+  (module Keybage_MountingHoles:MountingHole_2.2mm_M2_Pad_NoSilk (layer F.Cu)
+    (at 27.559 34.925)
+    (descr "Mounting Hole 2.2mm, M2, No Silk Ref")
+    (tags "mounting hole 2.2mm m2")
+    (attr virtual)
+    (fp_text reference U4 (at 0 -4) (layer F.SilkS) hide
+      (effects (font (size 1 1) (thickness 0.15)))
+    )
+    (fp_text value HOLE (at 0 0) (layer F.Fab)
+      (effects (font (size 1 1) (thickness 0.15)))
+    )
+    (fp_text user %R (at 0.3 0) (layer F.Fab)
+      (effects (font (size 1 1) (thickness 0.15)))
+    )
+    (fp_circle (center 0 0) (end 2.45 0) (layer F.CrtYd) (width 0.05))
+    (fp_circle (center 0 0) (end 2.2 0) (layer Cmts.User) (width 0.15))
+    (pad 1 thru_hole circle (at 0 0) (size 4.4 4.4) (drill 2.2) (layers *.Cu *.Mask))
+  )
+  (module Keybage_MountingHoles:MountingHole_2.2mm_M2_Pad_NoSilk (layer F.Cu)
+    (at 103.759 35.052)
+    (descr "Mounting Hole 2.2mm, M2, No Silk Ref")
+    (tags "mounting hole 2.2mm m2")
+    (attr virtual)
+    (fp_text reference U4 (at 0 -4) (layer F.SilkS) hide
+      (effects (font (size 1 1) (thickness 0.15)))
+    )
+    (fp_text value HOLE (at 0 0) (layer F.Fab)
+      (effects (font (size 1 1) (thickness 0.15)))
+    )
+    (fp_text user %R (at 0.3 0) (layer F.Fab)
+      (effects (font (size 1 1) (thickness 0.15)))
+    )
+    (fp_circle (center 0 0) (end 2.45 0) (layer F.CrtYd) (width 0.05))
+    (fp_circle (center 0 0) (end 2.2 0) (layer Cmts.User) (width 0.15))
+    (pad 1 thru_hole circle (at 0 0) (size 4.4 4.4) (drill 2.2) (layers *.Cu *.Mask))
+  )
+  (module Keybage_MountingHoles:MountingHole_2.2mm_M2_Pad_NoSilk (layer F.Cu)
+    (at 122.809 98.425)
+    (descr "Mounting Hole 2.2mm, M2, No Silk Ref")
+    (tags "mounting hole 2.2mm m2")
+    (attr virtual)
+    (fp_text reference U4 (at 0 -4) (layer F.SilkS) hide
+      (effects (font (size 1 1) (thickness 0.15)))
+    )
+    (fp_text value HOLE (at 0 0) (layer F.Fab)
+      (effects (font (size 1 1) (thickness 0.15)))
+    )
+    (fp_text user %R (at 0.3 0) (layer F.Fab)
+      (effects (font (size 1 1) (thickness 0.15)))
+    )
+    (fp_circle (center 0 0) (end 2.45 0) (layer F.CrtYd) (width 0.05))
+    (fp_circle (center 0 0) (end 2.2 0) (layer Cmts.User) (width 0.15))
+    (pad 1 thru_hole circle (at 0 0) (size 4.4 4.4) (drill 2.2) (layers *.Cu *.Mask))
+  )
+  (module Keybage_MountingHoles:MountingHole_2.2mm_M2_Pad_NoSilk (layer F.Cu)
+    (at 129.159 145.542)
+    (descr "Mounting Hole 2.2mm, M2, No Silk Ref")
+    (tags "mounting hole 2.2mm m2")
+    (attr virtual)
+    (fp_text reference U4 (at 0 -4) (layer F.SilkS) hide
+      (effects (font (size 1 1) (thickness 0.15)))
+    )
+    (fp_text value HOLE (at 0 0) (layer F.Fab)
+      (effects (font (size 1 1) (thickness 0.15)))
+    )
+    (fp_text user %R (at 0.3 0) (layer F.Fab)
+      (effects (font (size 1 1) (thickness 0.15)))
+    )
+    (fp_circle (center 0 0) (end 2.45 0) (layer F.CrtYd) (width 0.05))
+    (fp_circle (center 0 0) (end 2.2 0) (layer Cmts.User) (width 0.15))
+    (pad 1 thru_hole circle (at 0 0) (size 4.4 4.4) (drill 2.2) (layers *.Cu *.Mask))
+  )
+  (module Keybage_MountingHoles:MountingHole_2.2mm_M2_Pad_NoSilk (layer F.Cu)
+    (at 70.739 106.172)
+    (descr "Mounting Hole 2.2mm, M2, No Silk Ref")
+    (tags "mounting hole 2.2mm m2")
+    (attr virtual)
+    (fp_text reference U4 (at 0 -4) (layer F.SilkS) hide
+      (effects (font (size 1 1) (thickness 0.15)))
+    )
+    (fp_text value HOLE (at 0 0) (layer F.Fab)
+      (effects (font (size 1 1) (thickness 0.15)))
+    )
+    (fp_text user %R (at 0.3 0) (layer F.Fab)
+      (effects (font (size 1 1) (thickness 0.15)))
+    )
+    (fp_circle (center 0 0) (end 2.45 0) (layer F.CrtYd) (width 0.05))
+    (fp_circle (center 0 0) (end 2.2 0) (layer Cmts.User) (width 0.15))
+    (pad 1 thru_hole circle (at 0 0) (size 4.4 4.4) (drill 2.2) (layers *.Cu *.Mask))
+  )
+  (module Keybage_MountingHoles:MountingHole_2.2mm_M2_Pad_NoSilk (layer F.Cu)
+    (at 44.069 91.059)
+    (descr "Mounting Hole 2.2mm, M2, No Silk Ref")
+    (tags "mounting hole 2.2mm m2")
+    (attr virtual)
+    (fp_text reference U4 (at 0 -4) (layer F.SilkS) hide
+      (effects (font (size 1 1) (thickness 0.15)))
+    )
+    (fp_text value HOLE (at 0 0) (layer F.Fab)
+      (effects (font (size 1 1) (thickness 0.15)))
+    )
+    (fp_text user %R (at 0.3 0) (layer F.Fab)
+      (effects (font (size 1 1) (thickness 0.15)))
+    )
+    (fp_circle (center 0 0) (end 2.45 0) (layer F.CrtYd) (width 0.05))
+    (fp_circle (center 0 0) (end 2.2 0) (layer Cmts.User) (width 0.15))
+    (pad 1 thru_hole circle (at 0 0) (size 4.4 4.4) (drill 2.2) (layers *.Cu *.Mask))
   )
   (module SILK:mxnatee_med_back (layer B.Cu)
@@
       (xy -6.124192 -35.752678) (xy -5.173945 -35.835313) (xy -4.2545 -35.850498) (xy -3.515061 -35.833255)) (layer F.SilkS) (width 0.01))
   )
-  (module Keebio-Parts:MountingHole (layer F.Cu)
-    (at 103.759 35.052)
-    (fp_text reference U4 (at 0 -4) (layer F.SilkS) hide
-      (effects (font (size 1 1) (thickness 0.15)))
-    )
-    (fp_text value HOLE (at 0 0) (layer F.Fab)
-      (effects (font (size 1 1) (thickness 0.15)))
-    )
-    (fp_circle (center 0 0) (end 0 -2.8) (layer F.SilkS) (width 0.15))
-    (pad "" thru_hole circle (at 0 0) (size 6.5 6.5) (drill 6.5) (layers *.Cu *.Mask F.SilkS))
-  )
-  (module Keebio-Parts:MountingHole (layer F.Cu)
-    (at 122.809 98.425)
-    (fp_text reference U4 (at 0 -4) (layer F.SilkS) hide
-      (effects (font (size 1 1) (thickness 0.15)))
-    )
-    (fp_text value HOLE (at 0 0) (layer F.Fab)
-      (effects (font (size 1 1) (thickness 0.15)))
-    )
-    (fp_circle (center 0 0) (end 0 -2.8) (layer F.SilkS) (width 0.15))
-    (pad "" thru_hole circle (at 0 0) (size 6.5 6.5) (drill 6.5) (layers *.Cu *.Mask F.SilkS))
-  )
-  (module Keebio-Parts:MountingHole (layer F.Cu)
-    (at 129.159 145.542)
-    (fp_text reference U4 (at 0 -4) (layer F.SilkS) hide
-      (effects (font (size 1 1) (thickness 0.15)))
-    )
-    (fp_text value HOLE (at 0 0) (layer F.Fab)
-      (effects (font (size 1 1) (thickness 0.15)))
-    )
-    (fp_circle (center 0 0) (end 0 -2.8) (layer F.SilkS) (width 0.15))
-    (pad "" thru_hole circle (at 0 0) (size 6.5 6.5) (drill 6.5) (layers *.Cu *.Mask F.SilkS))
-  )
-  (module Keebio-Parts:MountingHole (layer F.Cu)
-    (at 70.739 106.172)
-    (fp_text reference U4 (at 0 -4) (layer F.SilkS) hide
-      (effects (font (size 1 1) (thickness 0.15)))
-    )
-    (fp_text value HOLE (at 0 0) (layer F.Fab)
-      (effects (font (size 1 1) (thickness 0.15)))
-    )
-    (fp_circle (center 0 0) (end 0 -2.8) (layer F.SilkS) (width 0.15))
-    (pad "" thru_hole circle (at 0 0) (size 6.5 6.5) (drill 6.5) (layers *.Cu *.Mask F.SilkS))
-  )
-  (module Keebio-Parts:MountingHole (layer F.Cu)
-    (at 44.069 91.059)
-    (fp_text reference U4 (at 0 -4) (layer F.SilkS) hide
-      (effects (font (size 1 1) (thickness 0.15)))
-    )
-    (fp_text value HOLE (at 0 0) (layer F.Fab)
-      (effects (font (size 1 1) (thickness 0.15)))
-    )
-    (fp_circle (center 0 0) (end 0 -2.8) (layer F.SilkS) (width 0.15))
-    (pad "" thru_hole circle (at 0 0) (size 6.5 6.5) (drill 6.5) (layers *.Cu *.Mask F.SilkS))
-  )
-  (module Keebio-Parts:MountingHole (layer F.Cu)
-    (at 27.559 34.925)
-    (fp_text reference U4 (at 0 -4) (layer F.SilkS) hide
-      (effects (font (size 1 1) (thickness 0.15)))
-    )
-    (fp_text value HOLE (at 0 0) (layer F.Fab)
-      (effects (font (size 1 1) (thickness 0.15)))
-    )
-    (fp_circle (center 0 0) (end 0 -2.8) (layer F.SilkS) (width 0.15))
-    (pad "" thru_hole circle (at 0 0) (size 6.5 6.5) (drill 6.5) (layers *.Cu *.Mask F.SilkS))
-  )
   (gr_line (start 149.597631 140.20487) (end 149.555111 141.13078) (layer Edge.Cuts) (width 0.05))
