File: Plates/Back Plate/mxnatee_bot_plate.kicad_pcb (KiCad board)
At the start: 2 copper layers, 137.5 x 139.4 mm, 8 parts, among them U4 HOLE

Commit message: Update
Parts:
- removed the U4 at (122.8, 98.4)
