File: Plates/Switch Plate/mxnatee_switch_plate.kicad_pcb (KiCad board)
At the start: 2 copper layers, 137.5 x 139.4 mm, 25 parts, among them U4 HOLE

Commit message: Update
Parts:
- removed the U4 at (122.8, 98.4)
Other:
- outline, holes or cut-outs redrawn
Changed lines of the file:
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@@
   (general
     (thickness 1.6)
-    (drawings 141)
+    (drawings 111)
     (tracks 0)
     (zones 0)
-    (modules 25)
+    (modules 24)
     (nets 7)
   )
@@
       (padsonsilk false)
       (subtractmaskfromsilk true)
-      (outputformat 1)
+      (outputformat 3)
       (mirror false)
       (drillshape 0)
       (scaleselection 1)
-      (outputdirectory "gerbers/"))
+      (outputdirectory "switch_plate_gerbers/"))
   )
   (net 0 "")
@@
   )
   (module Keybage_MountingHoles:MountingHole_2.2mm_M2_Pad_NoSilk (layer F.Cu)
-    (at 122.809 98.425)
-    (descr "Mounting Hole 2.2mm, M2, No Silk Ref")
-    (tags "mounting hole 2.2mm m2")
-    (attr virtual)
-    (fp_text reference U4 (at 0 -4) (layer F.SilkS) hide
-      (effects (font (size 1 1) (thickness 0.15)))
-    )
-    (fp_text value HOLE (at 0 0) (layer F.Fab)
-      (effects (font (size 1 1) (thickness 0.15)))
-    )
-    (fp_text user %R (at 0.3 0) (layer F.Fab)
-      (effects (font (size 1 1) (thickness 0.15)))
-    )
-    (fp_circle (center 0 0) (end 2.45 0) (layer F.CrtYd) (width 0.05))
-    (fp_circle (center 0 0) (end 2.2 0) (layer Cmts.User) (width 0.15))
-    (pad 1 thru_hole circle (at 0 0) (size 4.4 4.4) (drill 2.2) (layers *.Cu *.Mask))
-  )
-  (module Keybage_MountingHoles:MountingHole_2.2mm_M2_Pad_NoSilk (layer F.Cu)
     (at 129.159 145.542)
     (descr "Mounting Hole 2.2mm, M2, No Silk Ref")
@@
     (pad 1 thru_hole circle (at 0 0) (size 4.4 4.4) (drill 2.2) (layers *.Cu *.Mask))
   )
+  (gr_line (start 112.962043 28.645592) (end 113.351624 28.836688) (layer Edge.Cuts) (width 0.05))
+  (gr_line (start 142.418547 105.719035) (end 142.87 103.92) (layer Edge.Cuts) (width 0.05))
+  (gr_line (start 113.34 103.92) (end 142.87 103.92) (layer Edge.Cuts) (width 0.05))
+  (gr_line (start 113.35 46.77) (end 113.34 103.92) (layer Edge.Cuts) (width 0.05))
+  (gr_line (start 113.35 46.77) (end 113.35 28.84) (layer Edge.Cuts) (width 0.05))
   (gr_line (start 149.597631 140.20487) (end 149.555111 141.13078) (layer Edge.Cuts) (width 0.05))
-  (gr_line (start 145.814461 87.146364) (end 145.649594 88.909214) (layer Edge.Cuts) (width 0.05))
   (gr_line (start 148.276518 133.355524) (end 148.608387 134.339858) (layer Edge.Cuts) (width 0.05))
   (gr_line (start 147.1281 130.465312) (end 147.536374 131.418251) (layer Edge.Cuts) (width 0.05))
-  (gr_line (start 145.761871 75.489573) (end 145.896289 77.080571) (layer Edge.Cuts) (width 0.05))
-  (gr_line (start 145.217467 92.490812) (end 144.950208 94.309561) (layer Edge.Cuts) (width 0.05))
-  (gr_line (start 145.168627 70.834775) (end 145.39804 72.366675) (layer Edge.Cuts) (width 0.05))
   (gr_curve (pts (xy 149.597631 140.20487) (xy 149.563183 139.252659) (xy 149.458472 138.282208) (xy 149.291073 137.301909)) (layer Edge.Cuts) (width 0.05))
   (gr_curve (pts (xy 149.291073 137.301909) (xy 149.123674 136.321609) (xy 148.893587 135.331462) (xy 148.608387 134.339858)) (layer Edge.Cuts) (width 0.05))
@@
   (gr_curve (pts (xy 147.1281 130.465312) (xy 146.690093 129.536497) (xy 146.230844 128.639936) (xy 145.758129 127.782899)) (layer Edge.Cuts) (width 0.05))
   (gr_curve (pts (xy 145.758129 127.782899) (xy 145.285414 126.925861) (xy 144.799231 126.108348) (xy 144.307355 125.337631)) (layer Edge.Cuts) (width 0.05))
-  (gr_curve (pts (xy 145.39804 72.366675) (xy 145.579955 73.928124) (xy 145.579955 73.928124) (xy 145.761871 75.489573)) (layer Edge.Cuts) (width 0.05))
-  (gr_curve (pts (xy 145.896289 77.080571) (xy 145.982149 78.70077) (xy 146.018658 80.349862) (xy 146.005218 82.027583)) (layer Edge.Cuts) (width 0.05))
-  (gr_curve (pts (xy 146.005218 82.027583) (xy 145.991778 83.705304) (xy 145.928391 85.411653) (xy 145.814461 87.146364)) (layer Edge.Cuts) (width 0.05))
-  (gr_curve (pts (xy 145.649594 88.909214) (xy 145.43353 90.700013) (xy 145.43353 90.700013) (xy 145.217467 92.490812)) (layer Edge.Cuts) (width 0.05))
   (gr_line (start 143.816838 124.620122) (end 144.307355 125.337631) (layer Edge.Cuts) (width 0.05))
-  (gr_curve (pts (xy 144.207391 66.420074) (xy 144.571809 67.86106) (xy 144.892776 69.332773) (xy 145.168627 70.834775)) (layer Edge.Cuts) (width 0.05))
-  (gr_curve (pts (xy 144.950208 94.309561) (xy 144.631493 96.156073) (xy 144.261198 98.030196) (xy 143.839272 99.931814)) (layer Edge.Cuts) (width 0.05))
   (gr_line (start 55.3085 94.2975) (end 55.8165 93.2815) (layer Edge.Cuts) (width 0.05))
   (gr_line (start 54.356 95.758) (end 55.3085 94.2975) (layer Edge.Cuts) (width 0.05))
@@
   (gr_line (start 140.58459 111.724871) (end 139.904436 113.763137) (layer Edge.Cuts) (width 0.05))
   (gr_line (start 142.418547 105.719035) (end 141.841646 107.70282) (layer Edge.Cuts) (width 0.05))
-  (gr_line (start 142.49602 60.842291) (end 142.985451 62.189734) (layer Edge.Cuts) (width 0.05))
-  (gr_line (start 140.878215 56.928676) (end 141.442402 58.211762) (layer Edge.Cuts) (width 0.05))
-  (gr_line (start 136.18717 48.751207) (end 136.923519 49.830737) (layer Edge.Cuts) (width 0.05))
-  (gr_line (start 133.907807 45.656137) (end 134.679314 46.663907) (layer Edge.Cuts) (width 0.05))
-  (gr_line (start 128.323437 39.494612) (end 129.123805 40.277555) (layer Edge.Cuts) (width 0.05))
-  (gr_line (start 125.95134 37.297677) (end 126.737204 38.004673) (layer Edge.Cuts) (width 0.05))
-  (gr_line (start 120.795403 33.231053) (end 121.486202 33.721587) (layer Edge.Cuts) (width 0.05))
-  (gr_line (start 118.801348 31.88517) (end 119.452976 32.312844) (layer Edge.Cuts) (width 0.05))
-  (gr_line (start 114.639164 29.48565) (end 115.202553 29.7794) (layer Edge.Cuts) (width 0.05))
-  (gr_line (start 112.962043 28.645592) (end 113.518909 28.918747) (layer Edge.Cuts) (width 0.05))
   (gr_line (start 108.875715 26.756035) (end 109.497929 27.037516) (layer Edge.Cuts) (width 0.05))
   (gr_line (start 106.919954 25.874457) (end 107.586728 26.174505) (layer Edge.Cuts) (width 0.05))
@@
   (gr_line (start 139.420278 120.078872) (end 139.790913 120.274992) (layer Edge.Cuts) (width 0.05))
   (gr_line (start 138.397111 119.774809) (end 138.723377 119.82878) (layer Edge.Cuts) (width 0.05))
-  (gr_curve (pts (xy 138.987475 53.27799) (xy 139.647697 54.461191) (xy 140.27905 55.678296) (xy 140.878215 56.928676)) (layer Edge.Cuts) (width 0.05))
-  (gr_curve (pts (xy 136.923519 49.830737) (xy 137.638162 50.945495) (xy 138.327253 52.09479) (xy 138.987475 53.27799)) (layer Edge.Cuts) (width 0.05))
-  (gr_curve (pts (xy 134.679314 46.663907) (xy 135.433242 47.707557) (xy 135.433242 47.707557) (xy 136.18717 48.751207)) (layer Edge.Cuts) (width 0.05))
-  (gr_curve (pts (xy 123.670353 35.4009) (xy 124.415275 35.996572) (xy 125.176337 36.628487) (xy 125.95134 37.297677)) (layer Edge.Cuts) (width 0.05))
-  (gr_curve (pts (xy 121.486202 33.721587) (xy 122.196648 34.245802) (xy 122.925431 34.805229) (xy 123.670353 35.4009)) (layer Edge.Cuts) (width 0.05))
-  (gr_curve (pts (xy 119.452976 32.312844) (xy 120.12419 32.771949) (xy 120.12419 32.771949) (xy 120.795403 33.231053)) (layer Edge.Cuts) (width 0.05))
-  (gr_curve (pts (xy 116.956379 30.764638) (xy 117.555214 31.114381) (xy 118.16924 31.486673) (xy 118.801348 31.88517)) (layer Edge.Cuts) (width 0.05))
-  (gr_curve (pts (xy 115.202553 29.7794) (xy 115.773898 30.087701) (xy 116.357543 30.414895) (xy 116.956379 30.764638)) (layer Edge.Cuts) (width 0.05))
-  (gr_curve (pts (xy 113.518909 28.918747) (xy 114.079036 29.202198) (xy 114.079036 29.202198) (xy 114.639164 29.48565)) (layer Edge.Cuts) (width 0.05))
   (gr_curve (pts (xy 111.263137 27.846397) (xy 111.838966 28.113246) (xy 112.403745 28.378482) (xy 112.962043 28.645592)) (layer Edge.Cuts) (width 0.05))
   (gr_curve (pts (xy 109.497929 27.037516) (xy 110.100429 27.311083) (xy 110.687308 27.579547) (xy 111.263137 27.846397)) (layer Edge.Cuts) (width 0.05))
@@
   (gr_curve (pts (xy 139.904436 113.763137) (xy 139.17269 115.82859) (xy 138.389397 117.921204) (xy 137.554559 120.040981)) (layer Edge.Cuts) (width 0.05))
   (gr_curve (pts (xy 141.841646 107.70282) (xy 141.213118 109.713846) (xy 141.213118 109.713846) (xy 140.58459 111.724871)) (layer Edge.Cuts) (width 0.05))
-  (gr_curve (pts (xy 143.839272 99.931814) (xy 143.417345 101.833432) (xy 142.943788 103.762545) (xy 142.418547 105.719035)) (layer Edge.Cuts) (width 0.05))
-  (gr_curve (pts (xy 142.985451 62.189734) (xy 143.435105 63.568828) (xy 143.842973 64.979087) (xy 144.207391 66.420074)) (layer Edge.Cuts) (width 0.05))
-  (gr_curve (pts (xy 141.442402 58.211762) (xy 141.969211 59.527026) (xy 141.969211 59.527026) (xy 142.49602 60.842291)) (layer Edge.Cuts) (width 0.05))
   (gr_curve (pts (xy 55.006076 16.022063) (xy 55.619461 16.02726) (xy 56.244342 16.031248) (xy 56.880719 16.03403)) (layer Edge.Cuts) (width 0.05))
   (gr_arc (start 40.651642 40.659965) (end 55.006076 16.022063) (angle -194.0299812) (layer Edge.Cuts) (width 0.05))
@@
   (gr_curve (pts (xy 97.058005 127.981447) (xy 96.698172 128.81743) (xy 96.698172 128.81743) (xy 96.338339 129.653413)) (layer Edge.Cuts) (width 0.05))
   (gr_curve (pts (xy 99.499813 124.565513) (xy 98.739194 125.430205) (xy 98.078652 126.287761) (xy 97.518189 127.138181)) (layer Edge.Cuts) (width 0.05))
-  (gr_curve (pts (xy 131.530099 42.854227) (xy 132.328857 43.750792) (xy 133.122851 44.684896) (xy 133.907807 45.656137)) (layer Edge.Cuts) (width 0.05))
-  (gr_curve (pts (xy 129.123805 40.277555) (xy 129.927818 41.098638) (xy 130.731341 41.957663) (xy 131.530099 42.854227)) (layer Edge.Cuts) (width 0.05))
-  (gr_curve (pts (xy 126.737204 38.004673) (xy 127.53032 38.749643) (xy 127.53032 38.749643) (xy 128.323437 39.494612)) (layer Edge.Cuts) (width 0.05))
   (zone (net 1) (net_name GND) (layer F.Cu) (hatch edge 0.508)
     (connect_pads (clearance 0.508))
